File: kicad/Amiga-HID_rev1.0/Amiga-HID_rev1.0.kicad_pcb (KiCad board)
At the start: 4 copper layers, 17 x 55 mm, 61 parts, among them J1 USB-A Host, J2 JST-XH-5A, J3 OLED I2C, J4 Reserve 3V3+GP+GND+VSYS, J5 JST-SH-3 SWD, J6 JST-SH-3 UART, J7 Conn_01x06_Pin, SW1 Boot, SW2 Run, U1 USBLC6-2SC6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

Commit message: fast fertig mit routing
Parts:
- removed the R3 at (161.6, 138.1)
- removed the R4 at (158.5, 140.4)
- moved R3 2.14 mm to (156.9, 139.5)
- moved C12 2.03 mm to (162.0, 128.4), turned to 0 degrees
- moved C19 1.99 mm to (162.0, 129.6), turned to 0 degrees
- moved C17 1.69 mm to (161.5, 123.7), turned to 90 degrees
- moved C10 1.40 mm to (156.8, 126.3), turned to 0 degrees
- moved R5 1.29 mm to (156.3, 124.6), turned to -90 degrees
- moved C11 1.22 mm to (157.9, 131.3)
- moved R6 1.21 mm to (156.9, 140.7), turned to 180 degrees
- moved C15 1.02 mm to (153.7, 131.8)
- moved C9 0.55 mm to (152.2, 127.9)
- moved R8 0.51 mm to (152.3, 129.8)
- moved R9 0.46 mm to (152.3, 128.8)
- moved C8 0.26 mm to (153.0, 127.0)
- moved L1 0.19 mm to (152.6, 125.2), turned to -90 degrees
- moved C6 0.17 mm to (162.7, 130.1)
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Connections:
- J2 pad 2: unconnected-(J2-Pin_2-Pad2) -> /GPIO7
- J4 pad 4: /GP_RES1 -> /GPIO8
- J4 pad 5: /GP_RES2 -> /GPIO9
- U1 pad 1: /USB_D+ -> /USB_DP
- U1 pad 2: GND -> unconnected-(U1-GND-Pad2)
- U1 pad 3: /USB_D- -> /USB_DM
- U1 pad 4: /USB_DM -> /USB_D-
- U1 pad 6: /USB_DP -> /USB_D+
- U4 pad 10: /GP_RES1 -> /GPIO7
- U4 pad 12: /GP_RES2 -> /GPIO8
Routing:
- net /SWDIO: track 0.00 -> 40.1 mm
- net /SWCLK: track 0.00 -> 39.5 mm
- net /QSPI_SS: track 0.00 -> 22.7 mm, vias 0 -> 1
- net /RUN: track 0.00 -> 19.9 mm, vias 0 -> 2
- net /KB_CLOCK_3V3: track 0.00 -> 19.7 mm
- net /KB_DATA_3V3: track 0.00 -> 17.3 mm
- net /QSPI_SD1: track 0.00 -> 15.6 mm
- net /LED2: track 0.87 -> 15.9 mm
- net /GPIO8: track 0.00 -> 14.2 mm, vias 0 -> 1
- net /KB_CLOCK_5V: track 0.00 -> 13.0 mm
- net /USB_DM: track 0.00 -> 12.6 mm
- net /QSPI_SD2: track 0.00 -> 12.4 mm
- net /GPIO9: track 0.00 -> 9.70 mm, vias 0 -> 1
- net /QSPI_SD3: track 0.00 -> 9.47 mm
- net /KB_DATA_5V: track 0.00 -> 8.40 mm
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