File: kicad/Amiga-HID_rev1.0/Amiga-HID_rev1.0.kicad_pcb (KiCad board)
At the start: 4 copper layers, 17 x 55 mm, 60 parts, among them J1 USB-A Host, J2 JST-XH-5A, J3 OLED I2C, J4 Reserve 3V3+GP+GND+VSYS, J5 JST-SH-3 SWD, J6 JST-SH-3 UART, J7 Conn_01x06_Pin, SW1 Boot, SW2 Run, U1 USBLC6-2SC6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

Commit message: J6 war spiegelverkehrt
Connections:
- J2 pad 1: /KB_CLOCK_5V -> GND
- J2 pad 2: /GPIO7 -> +5V_AMIGA
- J2 pad 4: +5V_AMIGA -> /GPIO7
- J2 pad 5: GND -> /KB_CLOCK_5V
Routing:
- net /KB_CLOCK_5V: track 13.0 -> 10.9 mm
- net +5V_AMIGA: track 44.5 -> 46.5 mm
- net /GPIO7: track 25.1 -> 27.1 mm
Changed lines of the file:
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@@
 		(tags "VSSOP SO JEDEC-MO-187-CA Texas_DCU0008A")
 		(property "Reference" "U5"
-			(at 0 -1.95 90)
+			(at -2.75 0 180)
 			(layer "F.SilkS")
 			(effects
@@
 		(tags "QFN DFN_QFN")
 		(property "Reference" "U4"
-			(at 4.62 -3.24 0)
+			(at -3.4425 -4.72 0)
 			(layer "F.SilkS")
 			(effects
@@
 			(remove_unused_layers no)
 			(roundrect_rratio 0.147059)
-			(net "/KB_CLOCK_5V")
+			(net "GND")
 			(pinfunction "Pin_1_1")
 			(pintype "passive")
@@
 			(layers "*.Cu" "*.Mask")
 			(remove_unused_layers no)
-			(net "/GPIO7")
+			(net "+5V_AMIGA")
 			(pinfunction "Pin_2_2")
 			(pintype "passive")
@@
 			(layers "*.Cu" "*.Mask")
 			(remove_unused_layers no)
-			(net "+5V_AMIGA")
+			(net "/GPIO7")
 			(pinfunction "Pin_4_4")
 			(pintype "passive")
@@
 			(layers "*.Cu" "*.Mask")
 			(remove_unused_layers no)
-			(net "GND")
+			(net "/KB_CLOCK_5V")
 			(pinfunction "Pin_5_5")
 			(pintype "passive")
@@
 	)
 	(gr_text "SDA"
+		(at 162.65 111.08 0)
+		(layer "F.SilkS")
+		(effects
+			(font
+				(size 0.8 0.8)
+				(thickness 0.12)
+			)
+		)
+	)
+	(gr_text "SDA"
 		(at 162.65 113.62 0)
 		(layer "F.SilkS")
@@
 		)
 	)
-	(gr_text "GND"
-		(at 153.5 149.869998 90)
+	(gr_text "KBC"
+		(at 153.5 149.87 90)
 		(layer "F.SilkS")
 		(effects
@@
 		)
 	)
-	(gr_text "+5V"
-		(at 156 149.93 90)
+	(gr_text "GP7"
+		(at 156 149.88 90)
 		(layer "F.SilkS")
 		(effects
@@
 		)
 	)
-	(gr_text "GP7"
-		(at 161.07 149.88 90)
+	(gr_text "+5V"
+		(at 161.07 149.93 90)
 		(layer "F.SilkS")
 		(effects
@@
 		)
 	)
-	(gr_text "KBC"
-		(at 163.6 149.87 90)
+	(gr_text "GND"
+		(at 163.6 149.869998 90)
 		(layer "F.SilkS")
 		(effects
@@
 	)
 	(segment
-		(start 160.14 143.318248)
-		(end 160.14 148.84)
-		(width 0.15)
-		(layer "F.Cu")
-		(net "/KB_CLOCK_5V")
-	)
-	(segment
-		(start 160.14 148.84)
-		(end 163.5 152.2)
+		(start 158.25 144.524999)
+		(end 153.5 149.274999)
 		(width 0.15)
 		(layer "F.Cu")
@@
 	)
 	(segment
-		(start 158.455001 143.07)
-		(end 159.891752 143.07)
+		(start 158.25 143.9)
+		(end 158.25 143.275001)
 		(width 0.15)
 		(layer "F.Cu")
@@
 	)
 	(segment
-		(start 158.25 143.275001)
-		(end 158.455001 143.07)
+		(start 153.5 149.274999)
+		(end 153.5 152.2)
 		(width 0.15)
 		(layer "F.Cu")
@@
 	(segment
 		(start 158.25 143.9)
-		(end 158.25 143.275001)
-		(width 0.15)
-		(layer "F.Cu")
-		(net "/KB_CLOCK_5V")
-	)
-	(segment
-		(start 159.891752 143.07)
-		(end 160.14 143.318248)
+		(end 158.25 144.524999)
 		(width 0.15)
 		(layer "F.Cu")
@@
 	)
 	(segment
-		(start 161.85 132.38)
-		(end 163.5 134.03)
+		(start 163.5 144.7)
+		(end 156 152.2)
 		(width 0.15)
 		(layer "B.Cu")
@@
 	)
 	(segment
-		(start 163.5 134.03)
-		(end 163.5 149.7)
+		(start 161.85 132.38)
+		(end 163.5 134.03)
 		(width 0.15)
 		(layer "B.Cu")
@@
 	)
 	(segment
-		(start 163.5 149.7)
-		(end 161 152.2)
+		(start 163.5 134.03)
+		(end 163.5 144.7)
 		(width 0.15)
 		(layer "B.Cu")
@@
 	)
 	(segment
-		(start 154.42 117.32)
-		(end 154.42 116.082)
+		(start 150.55 141.75)
+		(end 161 152.2)
 		(width 0.5)
 		(layer "In2.Cu")
@@
 	)
 	(segment
-		(start 151.69 117.32)
-		(end 150.55 118.46)
+		(start 150.55 118.46)
+		(end 150.55 141.75)
 		(width 0.5)
 		(layer "In2.Cu")
@@
 	)
 	(segment
-		(start 150.55 146.75)
-		(end 156 152.2)
+		(start 154.42 117.32)
+		(end 154.42 116.082)
 		(width 0.5)
 		(layer "In2.Cu")
@@
 	)
 	(segment
-		(start 154.42 117.32)
-		(end 151.69 117.32)
+		(start 151.69 117.32)
+		(end 150.55 118.46)
 		(width 0.5)
 		(layer "In2.Cu")
@@
 	)
 	(segment
-		(start 150.55 118.46)
-		(end 150.55 146.75)
+		(start 154.42 117.32)
+		(end 151.69 117.32)
 		(width 0.5)
 		(layer "In2.Cu")
