File: kicad/Amiga-HID_rev1.0/Amiga-HID_rev1.0.kicad_sch (KiCad schematic)
At the start: 59 parts, among them J1 USB-A Host, J2 JST-XH-5A, J3 OLED I2C, J4 Reserve 3V3+GP+GND+VSYS, J5 JST-SH-3 SWD, J6 JST-SH-3 UART, J7 Conn_01x06_Pin, SW1 Boot, SW2 Run, U1 USBLC6-2SC6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

Commit message: BOm aktualisiert
Parts:
- C1: LCSC C19702 -> C89831
- C10: value 4.7u -> 4.7uF; LCSC C14663 -> C368809
- C11, C5: LCSC (none) -> C161530
- C12, C8, C9: value 4.7u -> 4.7uF; LCSC (none) -> C368809
- C13, C14, C15, C16, C17, C18, C19, C2, C20, C21, C22, C23, C4: LCSC C14663 -> C161530
- C3: LCSC (none) -> C45783
- C6: value 15p -> 15pF; LCSC (none) -> C441742
- C7: value 15p -> 15pF; LCSC C14663 -> C441742
- D1, D2, D3: LCSC C181276 -> C52287404
- F1: LCSC (none) -> C7202014
- J2: LCSC C157932 -> C7551124
- J3: LCSC (none) -> C52016392
- J4: LCSC (none) -> C225480
- J7: LCSC (none) -> C5372829
- L1: value 2.2u -> 3.3uH; LCSC C1046 -> C42411119
- LED1: LCSC (none) -> C965804
- LED2: LCSC (none) -> C72038
- R1, R2: LCSC (none) -> C21190
- R10, R11, R5: LCSC C25104 -> C25105
- R12, R13: LCSC (none) -> C25900
- R3: LCSC C25804 -> C25744
- R4, R6, R7: LCSC (none) -> C11702
- R8, R9: LCSC (none) -> C25100
- U1: LCSC C7480 -> C19170930
- U2: LCSC C6186 -> C2688239
- U5: LCSC C53411 -> C53434
- Y1: LCSC C9002 -> C3003246

Commit message: nicht bestückte Komponenten entfernt aus 3d-Ansicht
Parts:
- C1: LCSC C89831 -> C15850
- C4, C5: LCSC C161530 -> C1525
- C6, C7: LCSC C441742 -> C18164617
- D1, D2, D3: LCSC C52287404 -> C53114226
- U4: LCSC C42411118 -> C41378174
Changed lines of the file:
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@@
 			)
 		)
-		(property "LCSC" "C161530"
+		(property "LCSC" "C1525"
 			(at 0 0 0)
 			(hide yes)
@@
 			)
 		)
-		(property "LCSC" "C52287404"
+		(property "LCSC" "C53114226"
 			(at 80.01 78.74 0)
 			(hide yes)
@@
 			)
 		)
-		(property "LCSC" "C42411118"
+		(property "LCSC" "C41378174"
 			(at 0 0 0)
 			(hide yes)
@@
 			)
 		)
-		(property "LCSC" "C441742"
+		(property "LCSC" "C18164617"
 			(at 0 0 0)
 			(hide yes)
@@
 			)
 		)
-		(property "LCSC" "C52287404"
+		(property "LCSC" "C53114226"
 			(at 95.25 78.74 0)
 			(hide yes)
@@
 			)
 		)
-		(property "LCSC" "C52287404"
+		(property "LCSC" "C53114226"
 			(at 81.28 38.1 0)
 			(hide yes)
@@
 			)
 		)
-		(property "LCSC" "C161530"
+		(property "LCSC" "C1525"
 			(at 134.62 41.91 0)
 			(hide yes)
@@
 			)
 		)
-		(property "LCSC" "C89831"
+		(property "LCSC" "C15850"
 			(at 96.52 41.91 0)
 			(hide yes)
@@
 			)
 		)
-		(property "LCSC" "C441742"
+		(property "LCSC" "C18164617"
 			(at 0 0 0)
 			(hide yes)
