File: kicad/Amiga-HID_rev1.1/Amiga-HID_rev1.1.kicad_pcb (KiCad board)
At the start: 4 copper layers, 17 x 55 mm, 60 parts, among them J1 USB-A Host, J2 JST S5B-XH-A, J3 OLED I2C, J4 Reserve 3V3+GP+GND+VSYS, J5 JST-SH-3 SWD, J6 JST-SH-3 UART, J7 Conn_01x06_Pin, SW1 Boot, SW2 Run, U1 USBLC6-2SC6, U2 AMS1117-3.3, U3 W25Q16JVSSIQ, U4 RP2350_60QFN, U5 TXS0102DCUR, Y1 ABM8-272-T3_12MHz_10pF_50Ω

Commit message: Mark REV 1.1 ready to manufacture
Other:
- board text added: "GP25"
