File: kicad/Amiga-HID_rev1.1/Amiga-HID_rev1.1.kicad_sch (KiCad schematic)
At the start: 59 parts, among them J1 USB-A Host, J2 JST S5B-XH-A, J3 OLED I2C, J4 Reserve 3V3+GP+GND+VSYS, J5 JST-SH-3 SWD, J6 JST-SH-3 UART, J7 Conn_01x06_Pin, SW1 Boot, SW2 Run, U1 USBLC6-2SC6, U2 AMS1117-3.3, U3 W25Q16JVSSIQ, U4 RP2350_60QFN, U5 TXS0102DCUR, Y1 ABM8-272-T3_12MHz_10pF_50Ω

Commit message: Mark REV 1.1 ready to manufacture
Parts:
- C21, J3, J4, J5, J6, J7, U3: now not fitted
- R1, R2: value 330 -> 1k; LCSC C23138 -> C21190
Changed lines of the file:
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@@
 		(on_board yes)
 		(in_pos_files yes)
-		(dnp no)
+		(dnp yes)
 		(property "Reference" "U3"
 			(at 63.5 139.7 0)
@@
 		(on_board yes)
 		(in_pos_files yes)
-		(dnp no)
+		(dnp yes)
 		(property "Reference" "J5"
 			(at 210.82 242.57 0)
@@
 		(on_board yes)
 		(in_pos_files yes)
-		(dnp no)
+		(dnp yes)
 		(property "Reference" "J3"
 			(at 107.95 246.38 0)
@@
 		(on_board yes)
 		(in_pos_files yes)
-		(dnp no)
+		(dnp yes)
 		(property "Reference" "C21"
 			(at 315.341 68.6816 0)
@@
 			)
 		)
-		(property "Value" "330"
+		(property "Value" "1k"
 			(at 373.38 31.75 90)
 			(show_name no)
@@
 			)
 		)
-		(property "LCSC" "C23138"
+		(property "LCSC" "C21190"
 			(at 0 0 0)
 			(hide yes)
@@
 			)
 		)
-		(property "Value" "330"
+		(property "Value" "1k"
 			(at 373.38 45.72 90)
 			(show_name no)
@@
 			)
 		)
-		(property "LCSC" "C23138"
+		(property "LCSC" "C21190"
 			(at 0 0 0)
 			(hide yes)
@@
 		(on_board yes)
 		(in_pos_files yes)
-		(dnp no)
+		(dnp yes)
 		(property "Reference" "J6"
 			(at 210.82 261.62 0)
@@
 		(on_board yes)
 		(in_pos_files yes)
-		(dnp no)
+		(dnp yes)
 		(fields_autoplaced yes)
 		(property "Reference" "J7"
@@
 		(on_board yes)
 		(in_pos_files yes)
-		(dnp no)
+		(dnp yes)
 		(property "Reference" "J4"
 			(at 107.95 261.62 0)
